File: Sp_O2 Project/Sp02_Module.kicad_sch (KiCad schematic)
At the start: 14 parts, among them SW1 SW_Push, SW2 SW_Push, SW3 SW_Push, U1 MAX30102, U2 SSD1306

Commit message: Add files via upload
Parts:
- C1, C2, C3: footprint (none) -> Capacitor_THT:C_Disc_D4.7mm_W2.5mm_P5.00mm
- D1: footprint (none) -> LED_THT:LED_D5.0mm
- R1, R2, R3, R4: footprint (none) -> Resistor_THT:R_Axial_DIN0207_L6.3mm_D2.5mm_P7.62mm_Horizontal
- SW1, SW2, SW3: footprint (none) -> Button_Switch_THT:SW_PUSH_6mm
- U1: footprint (none) -> Sp02_stuff:MAX30102_Module
- U2: footprint (none) -> Sp02_stuff:SSD1306_Module
Connections:
- net +5V: no longer A1.29 (GND), A1.4 (GND), C1.2, C2.2, C3.2, D1.1 (K), SW1.1, SW2.1, SW3.1, U1.4 (GND), U2.1 (GND)
- new net GND: A1.29 (GND), A1.4 (GND), C1.2, C2.2, C3.2, D1.1 (K), SW1.1, SW2.1, SW3.1, U1.4 (GND), U2.1 (GND)
